Commit message: .
added phase variable in state and the derivative of it in action (in bhr8tcphase);
added some new rewards;
can learn correctly from scratch

File: resources/robots/BHR8TC/bhr8tc.urdf (robot description, URDF)
Before this commit: robot BHR8-TC, 12 links, 11 joints
Links:
- link lankle: geometry collision mesh filename=BHR8TC_STL/lanklepitch.stl; visual mesh filename=BHR8TC_STL/lanklepitch.stl scale=1 1 1
- link rankle: geometry collision mesh filename=BHR8TC_STL/ranklepitch.stl; visual mesh filename=BHR8TC_STL/ranklepitch.stl scale=1 1 1
Joints:
- joint leg1_left: limit lower=-3.14 upper=3.14 effort=100.0 velocity=100.0 -> lower=-0.35 upper=0.35 effort=100.0 velocity=10.0
- joint leg1_right: limit lower=-3.14 upper=3.14 effort=100.0 velocity=100.0 -> lower=-0.35 upper=0.35 effort=100.0 velocity=10.0
- joint leg2_left: limit lower=-3.14 upper=3.14 effort=100.0 velocity=100.0 -> lower=-0.35 upper=0.5 effort=100.0 velocity=10.0
- joint leg2_right: limit lower=-3.14 upper=3.14 effort=100.0 velocity=100.0 -> lower=-0.5 upper=0.35 effort=100.0 velocity=10.0
- joint leg3_left: limit lower=-3.14 upper=3.14 effort=100.0 velocity=100.0 -> lower=-1.4 upper=0.43 effort=300.0 velocity=15.0
- joint leg3_right: limit lower=-3.14 upper=3.14 effort=100.0 velocity=100.0 -> lower=-1.4 upper=0.43 effort=300.0 velocity=15.0
- joint leg4_left: limit lower=-3.14 upper=3.14 effort=100.0 velocity=100.0 -> lower=-0.08 upper=2.25 effort=300.0 velocity=15.0
- joint leg4_right: limit lower=-3.14 upper=3.14 effort=100.0 velocity=100.0 -> lower=-0.08 upper=2.25 effort=300.0 velocity=15.0
- joint leg5_left: limit lower=-3.14 upper=3.14 effort=100.0 velocity=100.0 -> lower=-1.1 upper=0.35 effort=200.0 velocity=15.0
- joint leg5_right: limit lower=-3.14 upper=3.14 effort=100.0 velocity=100.0 -> lower=-1.1 upper=0.35 effort=200.0 velocity=15.0
